File: hardware/nes_shell.kicad_pcb (KiCad board)
At the start: 4 copper layers, 99 x 45 mm, 34 parts, among them J1 USB_C_Receptacle_USB2.0, J2 Micro_SD_Card, Q3 S8050, SW1 SW_Push, SW2 SW_Push, SW3 SW_Push, SW4 SW_Push, SW5 SW_Push, SW6 SW_Push, SW7 SW_Push, SW8 SW_Push, SW9 SW_Push, U2 STM32H7B0VBTx, U8 REF3033, U9 RT9193-33GB, Y1 Crystal_GND24, Y3 Crystal

Commit message: 添加了一些待做
Parts:
- removed SW9: SW_Push, my_footprint:KEY-SMD_4P-L4.2-W3.4-P2.15-LS4.5-TL
- added U12: STM32G031G8Ux, Package_DFN_QFN:QFN-28_4x4mm_P0.5mm, F.Cu at (171.1, 101.4)
- added U13: ~, Package_DFN_QFN:QFN-24-1EP_4x4mm_P0.5mm_EP2.8x2.8mm, F.Cu at (214.7, 72.5)
