File: hardware/nes_shell.kicad_sch (KiCad schematic)
At the start: 75 parts, among them J1 USB_C_Receptacle_USB2.0, J2 Micro_SD_Card, Q1 SS9012, Q2 PDTC114ET, Q3 S8050, SW1 SW_Push, SW2 SW_Push, SW3 SW_Push, SW4 SW_Push, SW5 SW_Push, SW6 SW_Push, SW7 SW_Push, SW8 SW_Push, U1 STM32H743IIKx, U12 STM32G031G8Ux, U14 W25Q32JVZP, U2 STM32H7B0VBTx, U3 STM32F411CEUx, U4 STM32G474RETx, U5 STM32H723ZGIx, U6 STM32H723ZGTx, U7 STM32H7B0IBKxQ, U8 REF3033, U9 RT9193-33GB, Y1 Crystal_GND24, Y2 Crystal_GND24, Y3 Crystal

Commit message: 添加了一些待做
Parts:
- added U15: MPU6050, my_footprint:MPU6050, symbol my_symbol:MPU6050
Connections:
- net IPS_BLK: now also U2.4 (PE5)
- net IPS_CS: now also U2.3 (PE4)
- net IPS_DC: now also U2.2 (PE3)
- net IPS_RST: now also U2.98 (PE1)
- net IPS_SCL: now also U2.1 (PE2)
- net IPS_SDA: now also U2.5 (PE6)
- net LED: now reaches Q2.1 (B)
- net LED: now also U2.7 (PC13)
Other:
- note added: "FLASH"
- note added: "Hyper RAM"
- note added: "Speaker"
- note added: "USB"
- note added: "WiFi & BLE"
- note added: "主控"
- note added: "供电"
- note added: "输入控制"
- note added: "陀螺仪"
