File: hardware/nes_shell_2/nes_shell.kicad_pcb (KiCad board)
At the start: 4 copper layers, 99 x 45 mm, 35 parts, among them J1 USB_C_Receptacle_USB2.0, J2 Micro_SD_Card, Q3 S8050, SW1 SW_Push, SW2 SW_Push, SW3 SW_Push, SW4 SW_Push, SW5 SW_Push, SW6 SW_Push, SW7 SW_Push, SW8 SW_Push, U12 STM32G031G8Ux, U2 STM32H7B0VBTx, U8 REF3033, U9 RT9193-33GB, Y1 Crystal_GND24, Y3 Crystal

Commit message: 修改了游戏机的布局、添加了一些元件
Parts:
- added AE1: Antenna_Chip, RF_Antenna:Texas_SWRA117D_2.4GHz_Left, B.Cu at (52.6, 67.9)
- added H5: MountingHole, MountingHole:MountingHole_2.2mm_M2, F.Cu at (50.0, 92.5)
- added H6: MountingHole, MountingHole:MountingHole_2.2mm_M2, F.Cu at (50.0, 152.5)
- added H7: MountingHole, MountingHole:MountingHole_2.2mm_M2, F.Cu at (115.0, 92.5)
- added H8: MountingHole, MountingHole:MountingHole_2.2mm_M2, F.Cu at (115.0, 152.5)
- added J3: HDMI_A, Connector_HDMI:HDMI_A_Contact_Technology_HDMI-19APL2_Horizontal, F.Cu at (57.6, 106.9)
- added J4: Conn_01x20_MountingPin, Connector_FFC-FPC:TE_2-1734839-0_1x20-1MP_P0.5mm_Horizontal, B.Cu at (63.8, 80.3)
- added J5: Conn_01x20_MountingPin, Connector_FFC-FPC:TE_2-1734839-0_1x20-1MP_P0.5mm_Horizontal, B.Cu at (63.8, 92.2)
- added J6: Conn_01x20_MountingPin, Connector_FFC-FPC:TE_2-1734839-0_1x20-1MP_P0.5mm_Horizontal, B.Cu at (99.5, 80.3)
- added J7: Conn_01x20_MountingPin, Connector_FFC-FPC:TE_2-1734839-0_1x20-1MP_P0.5mm_Horizontal, B.Cu at (99.5, 92.2)
- added J8: DE15_Plug_HighDensity_MountingHoles, Connector_Dsub:DSUB-15-HD_Female_Horizontal_P2.29x1.98mm_EdgePinOffset3.03mm_Housed_MountingHolesOffset4.94mm, F.Cu at (44.2, 137.5)
- added U14: W25Q32JVZP, Package_SON:WSON-8-1EP_6x5mm_P1.27mm_EP3.4x4.3mm, B.Cu at (81.2, 76.1)
- added U15: MPU6050, my_footprint:MPU6050, F.Cu at (67.9, 145.7)
- added U16: RP2040, Package_DFN_QFN:QFN-56-1EP_7x7mm_P0.4mm_EP3.2x3.2mm, F.Cu at (69.8, 106.4)
- added U17: MAX9814, Package_DFN_QFN:DFN-14-1EP_3x3mm_P0.4mm_EP1.78x2.35mm, F.Cu at (110.1, 136.4)
- added Y2: Crystal_GND24, Crystal:Crystal_SMD_2016-4Pin_2.0x1.6mm, B.Cu at (56.3, 67.5)
- D3, D4, J1, J2, R6, R7, U9: moved to F.Cu
- U13: moved to B.Cu
- moved U13 157.6 mm to (57.5, 61.2), turned to 180 degrees
- moved SW4 124.3 mm to (61.0, 131.0), turned to 0 degrees
- moved SW1 122.8 mm to (56.0, 126.0)
- moved SW3 120.9 mm to (61.0, 121.0), turned to 0 degrees
- moved J1 118.1 mm to (95.7, 152.1)
- moved SW2 115.6 mm to (66.0, 126.0)
- moved D4 114.1 mm to (94.5, 142.0), turned to 0 degrees
- moved D3 113.8 mm to (94.5, 140.1), turned to 0 degrees
- moved SW5 110.0 mm to (80.0, 134.0), turned to 0 degrees
- moved R7 106.6 mm to (103.2, 144.0), turned to 0 degrees
- moved SW6 105.1 mm to (89.0, 134.0), turned to 0 degrees
- moved R6 102.7 mm to (103.2, 141.5), turned to 0 degrees
- moved U9 101.1 mm to (97.5, 144.0), turned to 0 degrees
- moved SW8 92.8 mm to (101.4, 128.2), turned to 45 degrees
- moved U12 85.7 mm to (85.9, 111.0)
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Connections:
- U2 pad 1: unconnected-(U2-PE2-Pad1) -> /IPS_SCL
- U2 pad 2: unconnected-(U2-PE3-Pad2) -> /IPS_DC
- U2 pad 3: unconnected-(U2-PE4-Pad3) -> /IPS_CS
- U2 pad 4: unconnected-(U2-PE5-Pad4) -> /IPS_BLK
- U2 pad 5: unconnected-(U2-PE6-Pad5) -> /IPS_SDA
- U2 pad 7: unconnected-(U2-PC13-Pad7) -> /LED
- U2 pad 98: unconnected-(U2-PE1-Pad98) -> /IPS_RST
Other:
- board size 99 x 45 mm -> 71 x 116 mm
