File: hardware/nes_shell_2/nes_shell.kicad_sch (KiCad schematic)
At the start: 76 parts, among them J1 USB_C_Receptacle_USB2.0, J2 Micro_SD_Card, Q1 SS9012, Q2 PDTC114ET, Q3 S8050, SW1 SW_Push, SW2 SW_Push, SW3 SW_Push, SW4 SW_Push, SW5 SW_Push, SW6 SW_Push, SW7 SW_Push, SW8 SW_Push, U1 STM32H743IIKx, U12 STM32G031G8Ux, U14 W25Q32JVZP, U15 MPU6050, U2 STM32H7B0VBTx, U3 STM32F411CEUx, U4 STM32G474RETx, U5 STM32H723ZGIx, U6 STM32H723ZGTx, U7 STM32H7B0IBKxQ, U8 REF3033, U9 RT9193-33GB, Y1 Crystal_GND24, Y2 Crystal_GND24, Y3 Crystal

Commit message: 修改了游戏机的布局、添加了一些元件
Parts:
- added AE1: Antenna_Chip, RF_Antenna:Texas_SWRA117D_2.4GHz_Left, symbol Device:Antenna_Chip
- added BT1: Battery_Cell, symbol Device:Battery_Cell
- added H5, H6, H7, H8: MountingHole, MountingHole:MountingHole_2.2mm_M2, symbol Mechanical:MountingHole
- added J3: HDMI_A, Connector_HDMI:HDMI_A_Contact_Technology_HDMI-19APL2_Horizontal, symbol Connector:HDMI_A
- added J4, J5, J6, J7: Conn_01x20_MountingPin, Connector_FFC-FPC:TE_2-1734839-0_1x20-1MP_P0.5mm_Horizontal, symbol Connector_Generic_MountingPin:Conn_01x20_MountingPin
- added J8: DE15_Plug_HighDensity_MountingHoles, Connector_Dsub:DSUB-15-HD_Female_Horizontal_P2.29x1.98mm_EdgePinOffset3.03mm_Housed_MountingHolesOffset4.94mm, symbol Connector:DE15_Plug_HighDensity_MountingHoles
- added LS1: Speaker, symbol Device:Speaker
- added MK1: Microphone_Condenser, symbol Device:Microphone_Condenser
- added U16: RP2040, Package_DFN_QFN:QFN-56-1EP_7x7mm_P0.4mm_EP3.2x3.2mm, symbol MCU_RaspberryPi:RP2040
- added U17: MAX9814, Package_DFN_QFN:DFN-14-1EP_3x3mm_P0.4mm_EP1.78x2.35mm, symbol Amplifier_Audio:MAX9814
Connections:
- new net: U16.1 (IOVDD), U16.10 (IOVDD), U16.22 (IOVDD), U16.33 (IOVDD), U16.42 (IOVDD), U16.49 (IOVDD)
- new net: U16.23 (DVDD), U16.50 (DVDD)
- new net: U17.11 (GND), U17.15 (GND), U17.4 (GND), U17.7 (GND)
Other:
- note added: "FPGA/RP2040 HDMI VGA OUT"
- moved on the sheet: C16, C17, C20, C21, C22, C23, C24, C25, C26, D3, D4, H1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
Changed lines of the file:
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@@
 	(generator "eeschema")
 	(generator_version "8.0")
-	(paper "A3")
+	(paper "A2")
 	(title_block
 		(title "STMH7B0 NES游戏机")
