File: hardware/nes_shell/nes_shell.kicad_sch (KiCad schematic)
At the start: 76 parts, among them J1 USB_C_Receptacle_USB2.0, J2 Micro_SD_Card, Q1 SS9012, Q2 PDTC114ET, Q3 S8050, SW1 SW_Push, SW2 SW_Push, SW3 SW_Push, SW4 SW_Push, SW5 SW_Push, SW6 SW_Push, SW7 SW_Push, SW8 SW_Push, U1 STM32H743IIKx, U12 STM32G031G8Ux, U14 W25Q32JVZP, U15 MPU6050, U2 STM32H7B0VBTx, U3 STM32F411CEUx, U4 STM32G474RETx, U5 STM32H723ZGIx, U6 STM32H723ZGTx, U7 STM32H7B0IBKxQ, U8 REF3033, U9 RT9193-33GB, Y1 Crystal_GND24, Y2 Crystal_GND24, Y3 Crystal

Commit message: 全新的分离设计，将不同的板子分在不同的项目当中
Parts:
- removed C13: 1uF, symbol Device:C_Polarized
- removed C18, C7, C8: C, symbol Device:C
- removed C5: 100nF, Capacitor_SMD:C_0402_1005Metric, symbol Device:C
- removed D1: BAT54C, Package_TO_SOT_SMD:SOT-23, symbol Diode:BAT54C
- removed D3, D4: ESD9B3.3ST5G, Diode_SMD:D_SOD-923, symbol Diode:ESD9B3.3ST5G
- removed FB1: FerriteBead, symbol Device:FerriteBead
- removed J1: USB_C_Receptacle_USB2.0, Connector_USB:USB_C_Receptacle_GCT_USB4105-xx-A_16P_TopMnt_Horizontal, symbol Connector:USB_C_Receptacle_USB2.0
- removed J2: Micro_SD_Card, Connector_Card:microSD_HC_Molex_47219-2001, symbol Connector:Micro_SD_Card
- removed Q3: S8050, Package_TO_SOT_SMD:SOT-23, symbol Transistor_BJT:S8050
- removed R10: 10k, symbol Device:R
- removed R6, R7: 5.1K, Resistor_SMD:R_0603_1608Metric, symbol Device:R
- removed R8: 10, symbol Device:R
- removed R9: 1k, symbol Device:R
- removed SW1, SW2, SW3, SW4, SW5, SW6, SW7, SW8: SW_Push, my_footprint:KEY-SMD_4P-L4.2-W3.4-P2.15-LS4.5-TL, symbol Switch:SW_Push
- removed U1: STM32H743IIKx, Package_BGA:UFBGA-201_10x10mm_Layout15x15_P0.65mm, symbol MCU_ST_STM32H7:STM32H743IIKx
- removed U10: ~, my_footprint:ips_2.0_240x320_12p, symbol my_symbol:ips_2.0_240x320_12P
- removed U11: ~, my_footprint:ns_joystick, symbol my_symbol:ns_joystick
- removed U12: STM32G031G8Ux, Package_DFN_QFN:QFN-28_4x4mm_P0.5mm, symbol MCU_ST_STM32G0:STM32G031G8Ux
- removed U13: ~, Package_DFN_QFN:QFN-24-1EP_4x4mm_P0.5mm_EP2.8x2.8mm, symbol my_chips:ESP8684
- removed U14: W25Q32JVZP, Package_SON:WSON-8-1EP_6x5mm_P1.27mm_EP3.4x4.3mm, symbol Memory_Flash:W25Q32JVZP
- removed U15: MPU6050, my_footprint:MPU6050, symbol my_symbol:MPU6050
- removed U2: STM32H7B0VBTx, Package_QFP:LQFP-100_14x14mm_P0.5mm, symbol MCU_ST_STM32H7:STM32H7B0VBTx
- removed U3: STM32F411CEUx, Package_DFN_QFN:QFN-48-1EP_7x7mm_P0.5mm_EP5.6x5.6mm, symbol MCU_ST_STM32F4:STM32F411CEUx
- removed U4: STM32G474RETx, Package_QFP:LQFP-64_10x10mm_P0.5mm, symbol MCU_ST_STM32G4:STM32G474RETx
- removed U5: STM32H723ZGIx, Package_BGA:UFBGA-144_7x7mm_Layout12x12_P0.5mm, symbol MCU_ST_STM32H7:STM32H723ZGIx
- removed U6: STM32H723ZGTx, Package_QFP:LQFP-144_20x20mm_P0.5mm, symbol MCU_ST_STM32H7:STM32H723ZGTx
- removed U7: STM32H7B0IBKxQ, Package_BGA:UFBGA-201_10x10mm_Layout15x15_P0.65mm, symbol MCU_ST_STM32H7:STM32H7B0IBKxQ
- removed U8: REF3033, Package_TO_SOT_SMD:SOT-23, symbol Reference_Voltage:REF3033
- removed U9: RT9193-33GB, Package_TO_SOT_SMD:SOT-23-5, symbol my_chips:RT9193-33GB
- removed Y2: Crystal_GND24, Crystal:Crystal_SMD_2016-4Pin_2.0x1.6mm, symbol Device:Crystal_GND24
- added C1: 1uF, symbol Device:C
- added C12, C13, C27, C28, C29: 0.1uF, Capacitor_SMD:C_0201_0603Metric, symbol Device:C
- added C2, C3, C4: 0.1u, symbol Device:C
- added C31, C32, C33: 2.2u, symbol Device:C
- added J1, J2: Conn_01x20_MountingPin, Connector_FFC-FPC:TE_2-1734839-0_1x20-1MP_P0.5mm_Horizontal, symbol Connector_Generic_MountingPin:Conn_01x20_MountingPin
- added J3, J4, J5, J6, J7: Conn_02x06_Odd_Even, Connector_PinSocket_1.27mm:PinSocket_2x06_P1.27mm_Vertical_SMD, symbol Connector_Generic:Conn_02x06_Odd_Even
- added U1: STM32H7B0IBKxQ, Package_BGA:UFBGA-201_10x10mm_Layout15x15_P0.65mm, symbol MCU_ST_STM32H7:STM32H7B0IBKxQ
- C10, C11, C19, C20, C21, C22, C23, C24, C25, C26, C9: value C -> 0.1uF; footprint (none) -> Capacitor_SMD:C_0201_0603Metric
- C14, C16, C17: footprint (none) -> Capacitor_SMD:C_0201_0603Metric
- C15: value 0.47uF -> 0.1uF; footprint (none) -> Capacitor_SMD:C_0201_0603Metric
- C8: renamed from C6; value C -> 0.1uF; footprint (none) -> Capacitor_SMD:C_0201_0603Metric
- R1: value 10k -> 10K; footprint Capacitor_SMD:C_0402_1005Metric -> (none)
- renumbered C2 to C18, C12 to C30, C1 to C5, C3 to C6, C4 to C7, D2 to D1, H3 to H2, H2 to H3, R5 to R2, R4 to R3, R3 to R4, R2 to R5, Y3 to Y2
Connections:
- net VCC is gone; now on net +3V3: C16.1, C17.1
- net +3V3: now also C10.1, C11.1, C14.1, C15.1, C19.1, C20.1, C21.1, C22.1, C23.1, C24.1, C25.1, C26.1, C8.1, C9.1, R1.1, C1.2, C12.1, C13.1, C27.1, C28.1, C29.1, U1.D11 (VDD), U1.E12 (VDD), U1.E15 (VDD50_USB), U1.E4 (VDD), U1.F13 (VDD33_USB), U1.G4 (VDD), U1.H12 (VDD), U1.K4 (VDD), U1.L12 (VDD), U1.M5 (VDD), U1.M9 (VDD)
- net BOOT0: now also U1.C5 (BOOT0); no longer R1.1
- net GND: now also C20.2, C21.2, C22.2, C23.2, C24.2, C25.2, C26.2, C1.1, C12.2, C13.2, C2.2, C27.2, C28.2, C29.2, C3.2, C31.2, C32.2, C33.2, C4.2, U1.A1 (VSS), U1.A15 (VSS), U1.C2 (VSS), U1.D10 (VSS), U1.D6 (VSS), U1.E1 (VSS), U1.F10 (VSS), U1.F12 (VSS), U1.F2 (VSSSMPS), U1.F6 (VSS), U1.F7 (VSS), U1.F8 (VSS), U1.F9 (VSS), U1.G10 (VSS), U1.G6 (VSS), U1.G7 (VSS), U1.G8 (VSS), U1.G9 (VSS), U1.H10 (VSS), U1.H6 (VSS), U1.H7 (VSS), U1.H8 (VSS), U1.H9 (VSS), U1.J10 (VSS), U1.J14 (VSS), U1.J6 (VSS), U1.J7 (VSS), U1.J8 (VSS), U1.J9 (VSS), U1.K10 (VSS), U1.K12 (VSS), U1.K2 (VSS), U1.K6 (VSS), U1.K7 (VSS), U1.K8 (VSS), U1.K9 (VSS), U1.M10 (VSS), U1.M6 (VSS), U1.N3 (VSSA), U1.R1 (VSS), U1.R15 (VSS); no longer R1.2
- net NRST: now also U1.L1 (NRST)
- net OSC32_IN: now also U1.D2 (PC14)
- net OSC32_OUT: now also U1.D1 (PC15)
- net OSC_IN: now also U1.J1 (PH0)
- net OSC_OUT: now also U1.K1 (PH1)
- net VBAT: now also U1.E2 (VBAT)
- net VDD: no longer C10.1, C11.1, C15.1, C8.1, C9.1
- net VDDA: now also U1.M4 (VDDA); no longer C14.1
- net VREF+: now also U1.M3 (VREF+)
- new net: C33.1, U1.R13 (VCAP)
- new net: R1.2, U1.D4 (PDR_ON)
- new net: C31.1, U1.A4 (VCAP)
- new net: C32.1, U1.A14 (VCAP)
- new net +1V8: C2.1, C3.1, C4.1, U1.A13 (VDDLDO), U1.A3 (VDDLDO), U1.R14 (VDDLDO)
- new net DEBUG_JTCK-SWCLK: U1.B13 (PA13)
- new net DEBUG_JTDI: U1.A11 (PA15)
- new net DEBUG_JTDO-SWO: U1.A6 (PB3)
- new net DEBUG_JTMS-SWDIO: U1.A12 (PA14)
- new net DEBUG_JTRST: U1.B6 (PB4)
- new net VREF-: U1.L4 (VREF-)
- no-connect marks 2 -> 0
Other:
- added sheet MPU9250 (mpu9250.kicad_sch)
- added sheet PMOD接口 (pmods.kicad_sch)
- added sheet QSPI_Flash (qspi_flash.kicad_sch)
- added sheet SDRAM (sdram.kicad_sch)
- added sheet USB通信 (usb_communication.kicad_sch)
- added sheet 按键部分 (key_input.kicad_sch)
- added sheet 电源管理 (power_control.kicad_sch)
- added sheet 音视频输入输出 (media_inout.kicad_sch)
- note added: "1uF靠近VDD33USB引脚"
- note added: "H743在VOS0(480MHz)工况下，核心电压为1.38V， VDDLDO最小输入电压为1.62V,此处使用1.8V作为VDDLDO的输入电压， 相比3.3V，在满足CPU供电的同时，尽量降低LDO的压差， 可以大大江都芯片的发热和功耗"
- note added: "上板框机械孔"
- note added: "供电去耦"
- note added: "时钟"
- note added: "电源管理"
- note removed: "FLASH"
- note removed: "Hyper RAM"
- note removed: "Speaker"
- note removed: "USB"
- note removed: "WiFi & BLE"
- note removed: "供电"
- note removed: "芯片USB接口"
- note removed: "输入控制"
- note removed: "陀螺仪"
- company: (none) -> TheBadZhang
- title: STMH7B0 NES游戏机 -> STMH7B0掌上NES游戏机
- moved on the sheet: C18, C30, C5, C6, C7, C8, D1, H1, H2, H3, H4, Q1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
